File: KiCad/Schematic.kicad_sch (KiCad schematic)
At the start: 44 parts, among them U1 LMH6609MF, U2 LMH6609MF, U3 LMH6609MF, U4 LMH6609MF, U5 LMH6609MF, U6 LMH6609MF

Commit message: shematic uppdate
Connections:
- net at R14.1, R17.1, R20.1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: now also A1.5V_3 (+5V_3)
- net at R3.1, R6.1, R9.1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: now also A1.5V_2 (+5V_2), HC-05. (GND)
- net at R11.2: now also A1.1; no longer A1.7
- net at A1.0: now also HC-05. (GND)
- net at A1.6: no longer HC-05. (GND)
Other:
- note added: "Left Foot Loadcells + Amplifier"
- note added: "Right Foot Loadcells + Amplifier"
- note removed: "Left Foot Loadcell Amplifier"
- note removed: "Right Foot Loadcell Amplifier"
- moved on the sheet: HC-05, TOF1
Changed lines of the file:
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@@
 	(text "Bluetooth Module"
 		(exclude_from_sim no)
-		(at 156.464 213.36 0)
+		(at 147.574 213.36 0)
 		(effects
 			(font
@@
 		)
 	)
-	(text "Right Foot Loadcell Amplifier"
+	(text "Right Foot Loadcells + Amplifier"
 		(exclude_from_sim no)
 		(at 294.64 26.67 0)
@@
 		)
 	)
-	(text "Left Foot Loadcell Amplifier"
+	(text "Left Foot Loadcells + Amplifier"
 		(exclude_from_sim no)
 		(at 125.476 25.654 0)
@@
 	)
 	(junction
+		(at 184.15 92.71)
+		(diameter 0)
+		(color 0 0 0 0)
+	)
+	(junction
 		(at 185.42 226.06)
 		(diameter 0)
@@
 	)
 	(junction
+		(at 184.15 180.34)
+		(diameter 0)
+		(color 0 0 0 0)
+	)
+	(junction
 		(at 317.5 60.96)
 		(diameter 0)
@@
 	(wire
 		(pts
-			(xy 171.45 222.25) (xy 200.66 222.25)
+			(xy 243.84 92.71) (xy 265.43 92.71)
 		)
 		(stroke
@@
 	(wire
 		(pts
-			(xy 243.84 92.71) (xy 265.43 92.71)
+			(xy 327.66 71.12) (xy 327.66 38.1)
 		)
 		(stroke
@@
 	(wire
 		(pts
-			(xy 327.66 71.12) (xy 327.66 38.1)
+			(xy 200.66 210.82) (xy 198.12 210.82)
 		)
 		(stroke
@@
 	(wire
 		(pts
-			(xy 274.32 168.91) (xy 274.32 241.3)
+			(xy 327.66 86.36) (xy 327.66 92.71)
+		)
+		(stroke
+			(width 0)
+			(type default)
+		)
+	)
+	(wire
+		(pts
+			(xy 274.32 165.1) (xy 274.32 241.3)
 		)
 		(stroke
@@
 	(wire
 		(pts
+			(xy 266.7 106.68) (xy 266.7 180.34)
+		)
+		(stroke
+			(width 0)
+			(type default)
+		)
+	)
+	(wire
+		(pts
 			(xy 349.25 81.28) (xy 349.25 77.47)
 		)
@@
 	(wire
 		(pts
+			(xy 162.56 229.87) (xy 177.8 229.87)
+		)
+		(stroke
+			(width 0)
+			(type default)
+		)
+	)
+	(wire
+		(pts
 			(xy 327.66 38.1) (xy 307.34 38.1)
 		)
@@
 	(wire
 		(pts
-			(xy 279.4 176.53) (xy 318.77 176.53)
+			(xy 279.4 172.72) (xy 316.23 172.72)
 		)
 		(stroke
@@
 	(wire
 		(pts
-			(xy 318.77 172.72) (xy 276.86 172.72)
+			(xy 316.23 168.91) (xy 276.86 168.91)
 		)
 		(stroke
@@
 	(wire
 		(pts
-			(xy 171.45 229.87) (xy 182.88 229.87)
-		)
-		(stroke
-			(width 0)
-			(type default)
-		)
-	)
-	(wire
-		(pts
 			(xy 171.45 38.1) (xy 171.45 39.37)
 		)
@@
 	(wire
 		(pts
-			(xy 279.4 190.5) (xy 279.4 176.53)
+			(xy 279.4 190.5) (xy 279.4 172.72)
 		)
 		(stroke
@@
 	(wire
 		(pts
+			(xy 327.66 106.68) (xy 266.7 106.68)
+		)
+		(stroke
+			(width 0)
+			(type default)
+		)
+	)
+	(wire
+		(pts
 			(xy 120.65 92.71) (xy 100.33 92.71)
 		)
@@
 	(wire
 		(pts
+			(xy 184.15 204.47) (xy 177.8 204.47)
+		)
+		(stroke
+			(width 0)
+			(type default)
+		)
+	)
+	(wire
+		(pts
 			(xy 242.57 49.53) (xy 252.73 49.53)
 		)
@@
 	(wire
 		(pts
-			(xy 182.88 229.87) (xy 182.88 180.34)
+			(xy 198.12 226.06) (xy 195.58 226.06)
 		)
 		(stroke
@@
 	(wire
 		(pts
-			(xy 274.32 168.91) (xy 318.77 168.91)
+			(xy 274.32 165.1) (xy 316.23 165.1)
 		)
 		(stroke
@@
 	(wire
 		(pts
+			(xy 177.8 229.87) (xy 177.8 204.47)
+		)
+		(stroke
+			(width 0)
+			(type default)
+		)
+	)
+	(wire
+		(pts
 			(xy 200.66 38.1) (xy 243.84 38.1)
 		)
@@
 	(wire
 		(pts
-			(xy 171.45 226.06) (xy 185.42 226.06)
+			(xy 162.56 226.06) (xy 185.42 226.06)
 		)
 		(stroke
@@
 	(wire
 		(pts
+			(xy 198.12 210.82) (xy 198.12 226.06)
+		)
+		(stroke
+			(width 0)
+			(type default)
+		)
+	)
+	(wire
+		(pts
 			(xy 77.47 49.53) (xy 87.63 49.53)
 		)
@@
 	(wire
 		(pts
-			(xy 285.75 92.71) (xy 265.43 92.71)
+			(xy 265.43 92.71) (xy 285.75 92.71)
 		)
 		(stroke
@@
 	(wire
 		(pts
-			(xy 276.86 172.72) (xy 276.86 195.58)
+			(xy 276.86 168.91) (xy 276.86 195.58)
 		)
 		(stroke
@@
 	(wire
 		(pts
+			(xy 181.61 222.25) (xy 181.61 208.28)
+		)
+		(stroke
+			(width 0)
+			(type default)
+		)
+	)
+	(wire
+		(pts
 			(xy 274.32 241.3) (xy 254 241.3)
 		)
@@
 	(wire
 		(pts
+			(xy 241.3 180.34) (xy 266.7 180.34)
+		)
+		(stroke
+			(width 0)
+			(type default)
+		)
+	)
+	(wire
+		(pts
 			(xy 109.22 246.38) (xy 185.42 246.38)
 		)
@@
 	(wire
 		(pts
-			(xy 318.77 165.1) (xy 274.32 165.1)
+			(xy 316.23 161.29) (xy 274.32 161.29)
 		)
 		(stroke
@@
 	(wire
 		(pts
-			(xy 252.73 38.1) (xy 265.43 38.1)
+			(xy 184.15 92.71) (xy 184.15 180.34)
 		)
 		(stroke
@@
 	(wire
 		(pts
-			(xy 182.88 180.34) (xy 200.66 180.34)
+			(xy 252.73 38.1) (xy 265.43 38.1)
 		)
 		(stroke
@@
 	(wire
 		(pts
+			(xy 184.15 180.34) (xy 200.66 180.34)
+		)
+		(stroke
+			(width 0)
+			(type default)
+		)
+	)
+	(wire
+		(pts
 			(xy 336.55 60.96) (xy 336.55 49.53)
 		)
@@
 	(wire
 		(pts
-			(xy 195.58 226.06) (xy 200.66 226.06)
+			(xy 181.61 208.28) (xy 200.66 208.28)
+		)
+		(stroke
+			(width 0)
+			(type default)
+		)
+	)
+	(wire
+		(pts
+			(xy 184.15 180.34) (xy 184.15 204.47)
 		)
 		(stroke
@@
 	(wire
 		(pts
+			(xy 327.66 92.71) (xy 327.66 106.68)
+		)
+		(stroke
+			(width 0)
+			(type default)
+		)
+	)
+	(wire
+		(pts
 			(xy 327.66 38.1) (xy 336.55 38.1)
 		)
@@
 	(wire
 		(pts
-			(xy 274.32 165.1) (xy 274.32 137.16)
+			(xy 274.32 161.29) (xy 274.32 137.16)
 		)
 		(stroke
@@
 	(wire
 		(pts
-			(xy 327.66 86.36) (xy 327.66 92.71)
-		)
-		(stroke
-			(width 0)
-			(type default)
-		)
-	)
-	(wire
-		(pts
 			(xy 275.59 78.74) (xy 275.59 60.96)
 		)
@@
 	(wire
 		(pts
-			(xy 171.45 233.68) (xy 185.42 233.68)
+			(xy 162.56 233.68) (xy 185.42 233.68)
 		)
 		(stroke
@@
 	(wire
 		(pts
+			(xy 162.56 222.25) (xy 181.61 222.25)
+		)
+		(stroke
+			(width 0)
+			(type default)
+		)
+	)
+	(wire
+		(pts
 			(xy 294.64 38.1) (xy 307.34 38.1)
 		)
@@
 	(symbol
 		(lib_id "ProjectSymbols:Bluetooth_Module_HC-05")
-		(at 153.67 228.6 90)
+		(at 144.78 228.6 90)
 		(mirror x)
 		(unit 1)
@@
 		(dnp no)
 		(property "Reference" "HC-05"
-			(at 153.162 227.33 90)
+			(at 144.272 227.33 90)
 			(effects
 				(font
@@
 		)
 		(property "Value" "~"
-			(at 154.94 237.49 90)
+			(at 146.05 237.49 90)
 			(effects
 				(font
@@
 		)
 		(property "Footprint" ""
-			(at 153.67 228.6 0)
+			(at 144.78 228.6 0)
 			(effects
 				(font
@@
 		)
 		(property "Datasheet" ""
-			(at 153.67 228.6 0)
+			(at 144.78 228.6 0)
 			(effects
 				(font
@@
 		)
 		(property "Description" ""
-			(at 153.67 228.6 0)
+			(at 144.78 228.6 0)
 			(effects
 				(font
@@
 	(symbol
 		(lib_id "ProjectSymbols:Time_of_Flight_Distance_Sensor_VL53L0X")
-		(at 327.66 170.18 270)
+		(at 325.12 166.37 270)
 		(unit 1)
 		(exclude_from_sim no)
@@
 		(dnp no)
 		(property "Reference" "TOF1"
-			(at 329.184 170.688 90)
+			(at 326.644 166.878 90)
 			(effects
 				(font
@@
 		)
 		(property "Value" "~"
-			(at 336.55 172.085 90)
+			(at 334.01 168.275 90)
 			(effects
 				(font
@@
 		)
 		(property "Footprint" ""
-			(at 327.66 170.18 0)
+			(at 325.12 166.37 0)
 			(effects
 				(font
@@
 		)
 		(property "Datasheet" ""
-			(at 327.66 170.18 0)
+			(at 325.12 166.37 0)
 			(effects
 				(font
@@
 		)
 		(property "Description" ""
-			(at 327.66 170.18 0)
+			(at 325.12 166.37 0)
 			(effects
 				(font
